File: pspMidi.kicad_pcb (KiCad board)
At the start: 2 copper layers, 34 parts, among them J1 USB_C_Receptacle_USB2.0, J2 AVR-ISP-6, SW1 SW_Push, U1 ATmega32U4RC-MU, U2 CD74HC4067M, U3 CD74HC4067M, Y1 Crystal_GND2_Small

Commit message: V1 done
Parts:
- added REF**: MountingHole_3.2mm_M3, MountingHole:MountingHole_3.2mm_M3, F.Cu at (41.0, 56.0)
- added REF**: MountingHole_3.2mm_M3, MountingHole:MountingHole_3.2mm_M3, F.Cu at (41.0, 101.0)
- added REF**: MountingHole_3.2mm_M3, MountingHole:MountingHole_3.2mm_M3, F.Cu at (236.0, 101.0)
- added REF**: MountingHole_3.2mm_M3, MountingHole:MountingHole_3.2mm_M3, F.Cu at (236.0, 56.0)
- U1: value ATmega32U4RC-MU -> ATmega32U4-MU
- moved SW1 72.4 mm to (206.0, 95.5), turned to 0 degrees
- moved R5 54.6 mm to (209.5, 83.1), turned to 0 degrees
- moved D1 31.2 mm to (217.6, 99.6), turned to 270 degrees
- moved R6 30.4 mm to (215.9, 99.7), turned to 270 degrees
- moved D2 25.2 mm to (217.5, 95.3), turned to 90 degrees
- moved R7 24.7 mm to (215.9, 95.3), turned to 270 degrees
- moved J1 2.00 mm to (229.6, 58.7)
- moved R1 2.00 mm to (228.1, 61.8)
- moved R2 2.00 mm to (225.0, 61.9)
- moved R3 2.00 mm to (222.0, 61.8)
- moved R4 2.00 mm to (231.1, 61.8)
- moved C1 0.89 mm to (217.3, 86.3)
Routing:
- net Net-(U3-Pad19): track 0.00 -> 320.7 mm, vias 0 -> 1
- net Net-(U3-Pad21): track 0.00 -> 288.6 mm, vias 0 -> 2
- net Net-(U3-Pad20): track 0.00 -> 276.6 mm, vias 0 -> 1
- net Net-(U3-Pad22): track 0.00 -> 265.3 mm, vias 0 -> 2
- net Net-(U3-Pad23): track 0.00 -> 241.0 mm, vias 0 -> 2
- net Net-(U3-Pad2): track 0.00 -> 207.8 mm
- net Net-(U3-Pad3): track 0.00 -> 186.0 mm
- net Net-(U3-Pad9): track 0.00 -> 141.8 mm, vias 0 -> 4
- net Net-(U3-Pad8): track 0.00 -> 108.7 mm, vias 0 -> 2
- net +5V: track 480.6 -> 573.2 mm, vias 0 -> 3
- net Net-(U3-Pad7): track 0.00 -> 71.1 mm, vias 0 -> 2
- net Net-(U1-Pad32): track 19.6 -> 84.5 mm, vias 1 -> 2
- net Net-(U3-Pad6): track 0.00 -> 55.1 mm
- net Net-(U1-Pad39): track 19.6 -> 63.2 mm, vias 1 -> 4
- net GND: track 180.7 -> 214.8 mm, vias 2 -> 23
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- added copper zone on B.Cu, net GND
- added copper zone on F.Cu, net GND
Other:
- board outline added: 203 x 53 mm
- board text added: "Raheel Rehmatullah pspMIDI January 2022"
