File: pspMidi.sch (KiCad schematic (older format))
At the start: 34 parts, among them J1 USB_C_Receptacle_USB2.0, J2 AVR-ISP-6, SW1 SW_Push, U1 ATmega32U4RC-MU, U2 CD74HC4067M, U3 CD74HC4067M, Y1 Crystal_GND2_Small

Commit message: V1 done
Parts:
- removed U1: ATmega32U4RC-MU, Package_DFN_QFN:QFN-44-1EP_7x7mm_P0.5mm_EP5.2x5.2mm, symbol MCU_Microchip_ATmega:ATmega32U4RC-MU
- added U1: ATmega32U4-MU, Package_DFN_QFN:QFN-44-1EP_7x7mm_P0.5mm_EP5.2x5.2mm, symbol MCU_Microchip_ATmega:ATmega32U4-MU
Connections:
- net +5V: now also U1.14 (VCC), U1.2 (UVCC), U1.24 (AVCC), U1.34 (VCC), U1.44 (AVCC), U1.7 (VBUS)
- net GND: now also U1.15 (GND), U1.23 (GND), U1.35 (GND), U1.43 (GND), U1.45 (GND), U1.5 (UGND)
- net RXLED: now also U1.8 (PB0)
- net TXLED: now also U1.22 (PD5)
- net at U2.1 (COM): now also U1.41 (PF0)
- net at U2.10 (S0), U3.10 (S0): now also U1.39 (PF4)
- net at U2.11 (S1), U3.11 (S1): now also U1.38 (PF5)
- net at U2.13 (S3), U3.13 (S3): now also U1.36 (PF7)
- net at U2.14 (S2), U3.14 (S2): now also U1.37 (PF6)
- net at U2.15 (~E), U3.15 (~E): now also U1.32 (PC7)
- net at U3.1 (COM): now also U1.40 (PF1)
- net at J2.4 (MOSI): now also U1.10 (PB2)
- net at J2.1 (MISO): now also U1.11 (PB3)
- net at J2.5 (~RST), R5.1, SW1.2: now also U1.13 (~RESET)
- net at C3.2, Y1.3: now also U1.16 (XTAL2)
- net at C2.1, Y1.1: now also U1.17 (XTAL1)
- net at R3.1: now also U1.3 (D-)
- net at R4.1: now also U1.4 (D+)
- net at C4.2: now also U1.42 (AREF)
- net at C1.2: now also U1.6 (UCAP)
- net at J2.3 (SCK): now also U1.9 (PB1)
